Commit message: visualisation and collision data added.

File: irp6_defs/robots/irp6p.urdf.xacro (robot description, xacro)
@@ -37,5 +37,5 @@
       <origin rpy="-1.57 0 0.0" xyz="0 0 0.4"/>
       <geometry>
-        <mesh filename="package://irp6_defs/meshes/link1.3ds" scale="0.01 0.01 0.01" />
+        <mesh filename="package://irp6_defs/meshes/link1.3ds" />
       </geometry>
     </visual>
@@ -63,5 +63,5 @@
       <origin rpy="0 0 0.0" xyz="0.45 0.0 0.0"/>
       <geometry>
-        <mesh filename="package://irp6_defs/meshes/link2.3ds" scale="0.01 0.01 0.01" />
+        <mesh filename="package://irp6_defs/meshes/link2.3ds" />
       </geometry>
     </visual>
@@ -89,11 +89,11 @@
       <origin rpy="0 0 1.57" xyz="0 0.67 0.0"/>
       <geometry>
-        <mesh filename="package://irp6_defs/meshes/link3.3ds" scale="0.01 0.01 0.01" />
+        <mesh filename="package://irp6_defs/meshes/link3.3ds" />
       </geometry>
     </visual>
     <collision>
-      <origin rpy="0 0 0.0" xyz="0 0.3 0.0"/>
+      <origin rpy="0 0 1.57" xyz="0 0.67 0.0"/>
       <geometry>
-        <box size="0.10 0.67 0.15"/>
+        <mesh filename="package://irp6_defs/meshes/link3.stlb" />
       </geometry>
     </collision>
@@ -115,7 +115,13 @@
       <origin rpy="1.57 0 1.57" xyz="0.0 0.175 0.0"/>
       <geometry>
-        <mesh filename="package://irp6_defs/meshes/link4.3ds" scale="0.01 0.01 0.01" />
+        <mesh filename="package://irp6_defs/meshes/link4.3ds" />
       </geometry>
     </visual>
+    <collision>
+      <origin rpy="1.57 0 1.57" xyz="0.0 0.175 0.0"/>
+      <geometry>
+        <mesh filename="package://irp6_defs/meshes/link4.stlb" />
+      </geometry>
+    </collision>
   </link>
   <joint name="joint5" type="revolute">
@@ -135,11 +141,11 @@
       <origin rpy="1.57 0 0.0" xyz="0.0 0.0 0.2"/>
       <geometry>
-        <mesh filename="package://irp6_defs/meshes/link5.3ds" scale="0.01 0.01 0.01" />
+        <mesh filename="package://irp6_defs/meshes/link5.3ds" />
       </geometry>
     </visual>
     <collision>
-      <origin rpy="1.57 0 0.0" xyz="0 0.12 0.2"/>
+      <origin rpy="1.57 0 0.0" xyz="0.0 0.0 0.2"/>
       <geometry>
-        <cylinder radius="0.05" length="0.30" />
+        <mesh filename="package://irp6_defs/meshes/link5.stlb" />
       </geometry>
     </collision>
@@ -161,5 +167,5 @@
       <origin rpy="0 0 0.0" xyz="0 0.0 0.0"/>
       <geometry>
-         <mesh filename="package://irp6_defs/meshes/link6.3ds" scale="0.01 0.01 0.01" />
+         <mesh filename="package://irp6_defs/meshes/link6.3ds" />
       </geometry>
     </visual>

Commit message: fix.

File: irp6_defs/robots/irp6p.urdf.xacro (robot description, xacro)
@@ -6,4 +6,23 @@
        xmlns:interface="http://playerstage.sourceforge.net/gazebo/xmlschema/#interface">
   <property name="M_PI" value="3.14159"/>
+  <link name="world">
+    <inertial>
+      <mass value="0.05" />
+      <origin xyz="-0.0 0.0 -10.0" />
+      <inertia ixx="1.0" ixy="0.0" ixz="0.0"
+               iyy="1.0" iyz="0.0"
+               izz="1.0" />
+    </inertial>
+    <collision>
+      <origin xyz="0 0 0.15" rpy="0 0 0" />
+      <geometry>
+        <box size="0.4 0.4 0.3" />
+      </geometry>
+    </collision>
+  </link>
+  <joint name="base_joint" type="fixed">
+    <parent link="world"/>
+    <child link="base_link"/>
+  </joint>
   <link name="base_link">
     <inertial>

File: irp6_launch/irp6p_fakeservo.xml.xacro (robot description, xacro)
@@ -112,6 +112,5 @@
 </struct>
 <struct name="JointTrajectoryAction" type="JointTrajectoryAction">
-  <struct name="Activity" type="PeriodicActivity">
- 	<simple name="Period" type="double"><value>0.1</value></simple>
+  <struct name="Activity" type="NonPeriodicActivity">
     <simple name="Priority" type="short"><value>2</value></simple>
     <simple name="Scheduler" type="string"><value>ORO_SCHED_RT</value></simple>

Commit message: new servo interface.

File: irp6_defs/robots/irp6p.urdf.xacro (robot description, xacro)
@@ -158,5 +158,5 @@
     </inertial>
     <visual>
-      <origin rpy="1.57 0 0.0" xyz="0.0 0.0 0.2"/>
+      <origin rpy="1.57 0 0.0" xyz="0.0 0.0 0.19"/>
       <geometry>
         <mesh filename="package://irp6_defs/meshes/link5.3ds" />
@@ -164,5 +164,5 @@
     </visual>
     <collision>
-      <origin rpy="1.57 0 0.0" xyz="0.0 0.0 0.2"/>
+      <origin rpy="1.57 0 0.0" xyz="0.0 0.0 0.19"/>
       <geometry>
         <mesh filename="package://irp6_defs/meshes/link5.stlb" />
@@ -171,5 +171,5 @@
   </link>
   <joint name="joint6" type="revolute">
-    <origin rpy="${0.5 * M_PI} 0 0" xyz="0.0 -0.1 0.2"/>
+    <origin rpy="${0.5 * M_PI} 0 0" xyz="0.0 -0.25 0.19"/>
     <axis xyz="0 0 1"/>
     <limit lower="0.0" upper="3.14" effort="10.0" velocity="10.0" />

Commit message: new interface fix.

File: irp6_defs/robots/irp6p.urdf.xacro (robot description, xacro)
@@ -60,7 +60,7 @@
     </visual>
     <collision>
-      <origin rpy="0 0 0.0" xyz="0 0 0.2"/>
-      <geometry>
-        <box size="0.22 0.25 0.4"/>
+      <origin rpy="-1.57 0 0.0" xyz="0 0 0.4"/>
+      <geometry>
+        <mesh filename="package://irp6_defs/meshes/link1.stlb" />
       </geometry>
     </collision>
@@ -69,5 +69,5 @@
     <origin rpy="${-0.5 * M_PI} 0 0" xyz="0.0 0.0 0.4"/>
     <axis xyz="0 0 1"/>
-    <limit lower="-2.26892803" upper="-0.872664626" effort="10.0" velocity="10.0" />
+    <limit lower="-1.8" upper="-0.872664626" effort="10.0" velocity="10.0" />
     <parent link="link1"/>
     <child link="link2"/>
@@ -95,5 +95,5 @@
     <origin rpy="0 0 0.0" xyz="0.45 0.0 0.0"/>
     <axis xyz="0 0 1"/>
-    <limit lower="-0.698131701" upper="0.698131701" effort="10.0" velocity="10.0" />
+    <limit lower="-0.3" upper="0.5" effort="10.0" velocity="10.0" />
     <parent link="link2"/>
     <child link="link3"/>
@@ -114,5 +114,5 @@
       <origin rpy="0 0 1.57" xyz="0 0.67 0.0"/>
       <geometry>
-        <mesh filename="package://irp6_defs/meshes/link3.stlb" />
+        <mesh filename="package://irp6_defs/meshes/link3.stlb" scale="1.0 1.0 1.3" />
       </geometry>
     </collision>
@@ -147,5 +147,5 @@
     <origin rpy="${-0.5 * M_PI} 0 0" xyz="0.0 0.0 0.0"/>
     <axis xyz="0 0 1"/>
-    <limit lower="0.0" upper="3.14" effort="10.0" velocity="10.0" />
+    <limit lower="-0.5" upper="5.14" effort="10.0" velocity="10.0" />
     <parent link="link4"/>
     <child link="link5"/>
@@ -171,7 +171,7 @@
   </link>
   <joint name="joint6" type="revolute">
-    <origin rpy="${0.5 * M_PI} 0 0" xyz="0.0 -0.25 0.19"/>
-    <axis xyz="0 0 1"/>
-    <limit lower="0.0" upper="3.14" effort="10.0" velocity="10.0" />
+    <origin rpy="${0.5 * M_PI} 0 0" xyz="0.0 -0.15 0.19"/>
+    <axis xyz="0 0 1"/>
+    <limit lower="-3.0" upper="2.9" effort="10.0" velocity="10.0" />
     <parent link="link5"/>
     <child link="link6"/>
@@ -190,10 +190,72 @@
     </visual>
     <collision>
-      <origin rpy="0.0 0 0.0" xyz="0 0.0 -0.04"/>
-      <geometry>
-        <cylinder radius="0.1" length="0.08" />
-      </geometry>
-    </collision>
-  </link>
+      <origin rpy="0.0 0 0.0" xyz="0 0.0 -0.05"/>
+      <geometry>
+        <cylinder radius="0.1" length="0.10" />
+      </geometry>
+    </collision>
+  </link>
+  <joint name="gripper_joint" type="fixed">
+    <origin rpy="0 0 0" xyz="0.0 0.0 0.06"/>
+    <parent link="link6"/>
+    <child link="griper_link"/>
+  </joint>
+  <link name="griper_link">
+    <inertial>
+      <mass value="0.1"/>
+      <origin xyz="0.0 0.0 0.0"/>
+      <inertia ixx="0.1" ixy="0" ixz="0" iyy="0.1" iyz="0" izz="0.1"/>
+    </inertial>
+    <visual>
+      <origin rpy="0 0 0.0" xyz="0 0.0 0.0"/>
+      <geometry>
+         <box size="0.05 0.1 0.12" />
+      </geometry>
+    </visual>
+    <collision>
+      <origin rpy="0.0 0 0.0" xyz="0 0.0 0.0"/>
+      <geometry>
+        <box size="0.05 0.2 0.12" />
+      </geometry>
+    </collision>
+  </link>
+<!-- Kinect                       -->
+<!--
+  <joint name="kinect_joint" type="fixed">
+    <origin rpy="0.0 0.87 1.58" xyz="0.715 -1.07 1.8"/>
+    <parent link="base_link"/>
+    <child link="kinect_base"/>
+  </joint>
+  <link name="kinect_base">
+  </link>
+  <joint name="kinect_depth_joint" type="fixed">
+    <origin rpy="0 0.0 0" xyz="0.0 -0.02 0.0"/>
+    <parent link="kinect_base"/>
+    <child link="openni_depth_frame"/>
+  </joint>
+  <link name="openni_depth_frame">
+  </link>
+  <joint name="kinect_rgb_joint" type="fixed">
+    <origin rpy="0 0.0 0" xyz="0.0 -0.04 0.0"/>
+    <parent link="kinect_base"/>
+    <child link="openni_rgb_frame"/>
+  </joint>
+  <link name="openni_rgb_frame">
+  </link>
+  <joint name="kinect_depth_optical_joint" type="fixed">
+    <origin xyz="0 0.0 0" rpy="1.57 0.0 1.57"/>
+    <parent link="openni_depth_frame"/>
+    <child link="openni_depth_optical_frame"/>
+  </joint>
+  <link name="openni_depth_optical_frame">
+  </link>
+  <joint name="kinect_rgb_optical_joint" type="fixed">
+    <origin xyz="0 0.0 0" rpy="1.57 0.0 1.57"/>
+    <parent link="openni_rgb_frame"/>
+    <child link="openni_rgb_optical_frame"/>
+  </joint>
+  <link name="openni_rgb_optical_frame">
+  </link>
+-->
 <!--
   <joint name="laser_tilt" type="revolute">
