Commit message: ...

File: irp6_description/robots/irp6p.urdf.xacro (robot description, xacro)
@@ -56,5 +56,5 @@
       <origin rpy="-1.57 0 0.0" xyz="0 0 0.4"/>
       <geometry>
-        <mesh filename="package://irp6_defs/meshes/link1.3ds" />
+        <mesh filename="package://irp6_description/meshes/link1.3ds" />
       </geometry>
     </visual>
@@ -62,5 +62,5 @@
       <origin rpy="-1.57 0 0.0" xyz="0 0 0.4"/>
       <geometry>
-        <mesh filename="package://irp6_defs/meshes/link1.stlb" />
+        <mesh filename="package://irp6_description/meshes/link1.stlb" />
       </geometry>
     </collision>
@@ -82,5 +82,5 @@
       <origin rpy="0 0 0.0" xyz="0.45 0.0 0.0"/>
       <geometry>
-        <mesh filename="package://irp6_defs/meshes/link2.3ds" />
+        <mesh filename="package://irp6_description/meshes/link2.3ds" />
       </geometry>
     </visual>
@@ -108,5 +108,5 @@
       <origin rpy="0 0 1.57" xyz="0 0.67 0.0"/>
       <geometry>
-        <mesh filename="package://irp6_defs/meshes/link3.3ds" />
+        <mesh filename="package://irp6_description/meshes/link3.3ds" />
       </geometry>
     </visual>
@@ -114,5 +114,5 @@
       <origin rpy="0 0 1.57" xyz="0 0.67 0.0"/>
       <geometry>
-        <mesh filename="package://irp6_defs/meshes/link3.stlb" scale="1.0 1.0 1.3" />
+        <mesh filename="package://irp6_description/meshes/link3.stlb" scale="1.0 1.0 1.3" />
       </geometry>
     </collision>
@@ -134,5 +134,5 @@
       <origin rpy="1.57 0 1.57" xyz="0.0 0.175 0.0"/>
       <geometry>
-        <mesh filename="package://irp6_defs/meshes/link4.3ds" />
+        <mesh filename="package://irp6_description/meshes/link4.3ds" />
       </geometry>
     </visual>
@@ -140,5 +140,5 @@
       <origin rpy="1.57 0 1.57" xyz="0.0 0.175 0.0"/>
       <geometry>
-        <mesh filename="package://irp6_defs/meshes/link4.stlb" />
+        <mesh filename="package://irp6_description/meshes/link4.stlb" />
       </geometry>
     </collision>
@@ -160,5 +160,5 @@
       <origin rpy="1.57 0 0.0" xyz="0.0 0.0 0.19"/>
       <geometry>
-        <mesh filename="package://irp6_defs/meshes/link5.3ds" />
+        <mesh filename="package://irp6_description/meshes/link5.3ds" />
       </geometry>
     </visual>
@@ -166,5 +166,5 @@
       <origin rpy="1.57 0 0.0" xyz="0.0 0.0 0.19"/>
       <geometry>
-        <mesh filename="package://irp6_defs/meshes/link5.stlb" />
+        <mesh filename="package://irp6_description/meshes/link5.stlb" />
       </geometry>
     </collision>
@@ -186,5 +186,5 @@
       <origin rpy="0 0 0.0" xyz="0 0.0 0.0"/>
       <geometry>
-         <mesh filename="package://irp6_defs/meshes/link6.3ds" />
+         <mesh filename="package://irp6_description/meshes/link6.3ds" />
       </geometry>
     </visual>

Commit message: kienatics fix due to rviz compatibility

File: irp6_description/robots/irp6p.urdf.xacro (robot description, xacro)
@@ -41,5 +41,5 @@
   </link>
   <joint name="joint1" type="revolute">
-    <origin rpy="0 0 0" xyz="0.0 0.0 0.3"/>
+    <origin rpy="0 0 0" xyz="0.0 0.0 0.55"/>
     <axis xyz="0 0 1"/>
     <limit lower="-2.96705973" upper="2.96705973" effort="10.0" velocity="10.0" />

Commit message: kineamtic fix

File: irp6_description/robots/irp6p.urdf.xacro (robot description, xacro)
@@ -93,5 +93,5 @@
   </link>
   <joint name="joint3" type="revolute">
-    <origin rpy="0 0 0.0" xyz="0.45 0.0 0.0"/>
+    <origin rpy="0 0 0.0" xyz="0.455 0.0 0.0"/>
     <axis xyz="0 0 1"/>
     <limit lower="-0.3" upper="0.5" effort="10.0" velocity="10.0" />
@@ -171,5 +171,5 @@
   </link>
   <joint name="joint6" type="revolute">
-    <origin rpy="${0.5 * M_PI} 0 0" xyz="0.0 -0.15 0.19"/>
+    <origin rpy="${0.5 * M_PI} 0 0" xyz="0.0 0.0 0.19"/>
     <axis xyz="0 0 1"/>
     <limit lower="-3.0" upper="2.9" effort="10.0" velocity="10.0" />
@@ -184,5 +184,5 @@
     </inertial>
     <visual>
-      <origin rpy="0 0 0.0" xyz="0 0.0 0.0"/>
+      <origin rpy="0 0 0.0" xyz="0 0.0 0.15"/>
       <geometry>
          <mesh filename="package://irp6_description/meshes/link6.3ds" />
@@ -197,5 +197,5 @@
   </link>
   <joint name="gripper_joint" type="fixed">
-    <origin rpy="0 0 0" xyz="0.0 0.0 0.06"/>
+    <origin rpy="0 0 0" xyz="0.0 0.0 0.21"/>
     <parent link="link6"/>
     <child link="griper_link"/>

Commit message: fix

File: irp6_description/robots/irp6p.urdf.xacro (robot description, xacro)
@@ -40,5 +40,5 @@
     </collision>
   </link>
-  <joint name="joint1" type="revolute">
+  <joint name="Irp6pmJoint1" type="revolute">
     <origin rpy="0 0 0" xyz="0.0 0.0 0.55"/>
     <axis xyz="0 0 1"/>
@@ -66,5 +66,5 @@
     </collision>
   </link>
-  <joint name="joint2" type="revolute">
+  <joint name="Irp6pmJoint2" type="revolute">
     <origin rpy="${-0.5 * M_PI} 0 0" xyz="0.0 0.0 0.4"/>
     <axis xyz="0 0 1"/>
@@ -92,5 +92,5 @@
     </collision>
   </link>
-  <joint name="joint3" type="revolute">
+  <joint name="Irp6pmJoint3" type="revolute">
     <origin rpy="0 0 0.0" xyz="0.455 0.0 0.0"/>
     <axis xyz="0 0 1"/>
@@ -118,5 +118,5 @@
     </collision>
   </link>
-  <joint name="joint4" type="revolute">
+  <joint name="Irp6pmJoint4" type="revolute">
     <origin rpy="0 0 0" xyz="0.0 0.67 0.0"/>
     <axis xyz="0 0 1"/>
@@ -144,5 +144,5 @@
     </collision>
   </link>
-  <joint name="joint5" type="revolute">
+  <joint name="Irp6pmJoint5" type="revolute">
     <origin rpy="${-0.5 * M_PI} 0 0" xyz="0.0 0.0 0.0"/>
     <axis xyz="0 0 1"/>
@@ -170,5 +170,5 @@
     </collision>
   </link>
-  <joint name="joint6" type="revolute">
+  <joint name="Irp6pmJoint6" type="revolute">
     <origin rpy="${0.5 * M_PI} 0 0" xyz="0.0 0.0 0.19"/>
     <axis xyz="0 0 1"/>
