Commit message: urdf fix

File: irp6_description/robots/irp6pboth.urdf.xacro (robot description, xacro)
@@ -210,5 +210,5 @@
   </link>
   <joint name="Irp6otmJoint7" type="revolute">
-    <origin rpy="1.570795 0 0" xyz="0.0 -0.15 0.19"/>
+    <origin rpy="1.570795 0 0" xyz="0.0 0.0 0.19"/>
     <axis xyz="0 0 1"/>
     <limit lower="-3.0" upper="2.9" effort="10.0" velocity="10.0" />
@@ -223,5 +223,5 @@
     </inertial>
     <visual>
-      <origin rpy="0 0 0.0" xyz="0 0.0 0.0"/>
+      <origin rpy="0 0 0.0" xyz="0 0.0 0.15"/>
       <geometry>
          <mesh filename="package://irp6_description/meshes/link6.3ds" />
@@ -236,5 +236,5 @@
   </link>
   <joint name="Irp6ottfgJoint1" type="prismatic">
-    <origin rpy="0 0 0" xyz="0.0 0.0 0.0"/>
+    <origin rpy="0 0 0" xyz="0.0 0.0 0.15"/>
     <parent link="link6"/>
     <child link="gripper_link_1"/>
@@ -243,5 +243,5 @@
   </joint>
   <joint name="Irp6ottfgJoint1a" type="prismatic">
-    <origin rpy="0 0 0" xyz="0.0 0.0 0.0"/>
+    <origin rpy="0 0 0" xyz="0.0 0.0 0.15"/>
     <parent link="link6"/>
     <child link="gripper_link_2"/>
@@ -441,5 +441,5 @@
   </link>
   <joint name="Irp6pmJoint6" type="revolute">
-    <origin rpy="1.570795 0 0" xyz="0.0 -0.15 0.19"/>
+    <origin rpy="1.570795 0 0" xyz="0.0 0.0 0.19"/>
     <axis xyz="0 0 1"/>
     <limit lower="-3.0" upper="2.9" effort="10.0" velocity="10.0" />
@@ -454,5 +454,5 @@
     </inertial>
     <visual>
-      <origin rpy="0 0 0.0" xyz="0 0.0 0.0"/>
+      <origin rpy="0 0 0.0" xyz="0 0.0 0.15"/>
       <geometry>
          <mesh filename="package://irp6_description/meshes/link6.3ds" />
@@ -467,5 +467,5 @@
   </link>
   <joint name="Irp6ptfgJoint1" type="prismatic">
-    <origin rpy="0 0 0" xyz="0.0 0.0 0.0"/>
+    <origin rpy="0 0 0" xyz="0.0 0.0 0.15"/>
     <parent link="link6_p"/>
     <child link="gripper_link_p_1"/>
@@ -474,5 +474,5 @@
   </joint>
   <joint name="Irp6ptfgJoint1a" type="prismatic">
-    <origin rpy="0 0 0" xyz="0.0 0.0 0.0"/>
+    <origin rpy="0 0 0" xyz="0.0 0.0 0.15"/>
     <parent link="link6_p"/>
     <child link="gripper_link_p_2"/>

Commit message: kinematic model cleanup

File: irp6_description/robots/irp6pboth.urdf.xacro (robot description, xacro)
@@ -74,5 +74,5 @@
   <parent link="base_link"/>
   <child link="postument"/>
-  <origin xyz="0 0 .01" rpy="0 0 0" />
+  <origin xyz="0 0 .25" rpy="0 0 0" />
   <axis xyz="0 1 0" />
   <limit upper="1.209" lower="0" effort="10" velocity=".53" />
@@ -119,5 +119,5 @@
     </inertial>
     <visual>
-      <origin rpy="0 0 0.0" xyz="0.45 0.0 0.0"/>
+      <origin rpy="0 0 0.0" xyz="0.455 0.0 0.0"/>
       <geometry>
         <mesh filename="package://irp6_description/meshes/link2.3ds" />
@@ -132,5 +132,5 @@
   </link>
   <joint name="Irp6otmJoint4" type="revolute">
-    <origin rpy="0 0 0.0" xyz="0.45 0.0 0.0"/>
+    <origin rpy="0 0 0.0" xyz="0.455 0.0 0.0"/>
     <axis xyz="0 0 1"/>
     <limit lower="-0.3" upper="0.5" effort="10.0" velocity="10.0" />
@@ -290,5 +290,5 @@
 <!-- -.-.-.-.-.-.-.-.-.-.-.-.-.-.-.-.-.-.-.-.-.-.-.-.-.-.-.-.-.-.-.-.-.-.-.-.-.-.-.-.-.-.- -->
   <joint name="base_joint_p" type="fixed">
-    <origin rpy="0 0 0" xyz="0.0 2.11 0.0"/>
+    <origin rpy="0 0 0.0" xyz="0.0 2.11 0.25"/>
     <parent link="world"/>
     <child link="base_link_p"/>
@@ -350,5 +350,5 @@
     </inertial>
     <visual>
-      <origin rpy="0 0 0.0" xyz="0.45 0.0 0.0"/>
+      <origin rpy="0 0 0.0" xyz="0.455 0.0 0.0"/>
       <geometry>
         <mesh filename="package://irp6_description/meshes/link2.3ds" />
@@ -363,5 +363,5 @@
   </link>
   <joint name="Irp6pmJoint3" type="revolute">
-    <origin rpy="0 0 0.0" xyz="0.45 0.0 0.0"/>
+    <origin rpy="0 0 0.0" xyz="0.455 0.0 0.0"/>
     <axis xyz="0 0 1"/>
     <limit lower="-0.3" upper="0.5" effort="10.0" velocity="10.0" />

Commit message: kinematic model cleanup

File: irp6_description/robots/irp6pboth.urdf.xacro (robot description, xacro)
@@ -32,7 +32,7 @@
   </inertial>
   <visual>
-    <origin xyz="0 .6045 .07" />
+    <origin xyz="0 .6045 .125" />
     <geometry>
-      <box size=".462 1.609 .2" />
+      <box size=".462 1.609 .25" />
     </geometry>
     <material name="gray">
@@ -55,7 +55,7 @@
   </inertial>
   <visual>
-    <origin xyz="0 0 0" />
+    <origin xyz="0 0 0.075" />
     <geometry>
-      <box size="-0.0 0.0 0.0" />
+      <box size="0.4 0.4 0.15" />
     </geometry>
     <material name="gray">
@@ -290,5 +290,5 @@
 <!-- -.-.-.-.-.-.-.-.-.-.-.-.-.-.-.-.-.-.-.-.-.-.-.-.-.-.-.-.-.-.-.-.-.-.-.-.-.-.-.-.-.-.- -->
   <joint name="base_joint_p" type="fixed">
-    <origin rpy="0 0 0.0" xyz="0.0 2.11 0.25"/>
+    <origin rpy="0 0 0.0" xyz="0.0 2.11 0.0"/>
     <parent link="world"/>
     <child link="base_link_p"/>
@@ -308,7 +308,16 @@
       </geometry>
     </collision>
+    <visual>
+      <origin xyz="0 0 0.2" />
+      <geometry>
+        <box size="0.4 0.4 0.4" />
+      </geometry>
+      <material name="gray">
+      <color rgba=".2 .2 .2 1" />
+    </material>
+  </visual>
   </link>
   <joint name="Irp6pmJoint1" type="revolute">
-    <origin rpy="0 0 0" xyz="0.0 0.0 0.3"/>
+    <origin rpy="0 0 0" xyz="0.0 0.0 0.55"/>
     <axis xyz="0 0 1"/>
     <limit lower="-2.96705973" upper="2.96705973" effort="10.0" velocity="10.0" />

Commit message: link names standarization

File: irp6_description/robots/irp6pboth.urdf.xacro (robot description, xacro)
@@ -23,7 +23,7 @@
   <joint name="base_joint" type="fixed">
     <parent link="world"/>
-    <child link="base_link"/>
-  </joint>
-<link name="base_link">
+    <child link="tl_base"/>
+  </joint>
+<link name="tl_base">
   <inertial>
     <mass value="1"/>
@@ -48,5 +48,5 @@
   </collision>
 </link>
-<link name="postument">
+<link name="tl_t">
   <inertial>
     <mass value="1"/>
@@ -72,6 +72,6 @@
 </link>
 <joint name="Irp6otmJoint1" type="prismatic">
-  <parent link="base_link"/>
-  <child link="postument"/>
+  <parent link="tl_base"/>
+  <child link="tl_t"/>
   <origin xyz="0 0 .25" rpy="0 0 0" />
   <axis xyz="0 1 0" />
@@ -82,8 +82,8 @@
     <axis xyz="0 0 1"/>
     <limit lower="-2.96705973" upper="2.96705973" effort="10.0" velocity="10.0" />
-    <parent link="postument"/>
-    <child link="link1"/>
-  </joint>
-  <link name="link1">
+    <parent link="tl_t"/>
+    <child link="tl_1"/>
+  </joint>
+  <link name="tl_1">
     <inertial>
       <mass value="0.1"/>
@@ -109,8 +109,8 @@
     <axis xyz="0 0 1"/>
     <limit lower="-1.8" upper="-0.872664626" effort="10.0" velocity="10.0" />
-    <parent link="link1"/>
-    <child link="link2"/>
-  </joint>
-  <link name="link2">
+    <parent link="tl_1"/>
+    <child link="tl_2"/>
+  </joint>
+  <link name="tl_2">
     <inertial>
       <mass value="0.1"/>
@@ -135,8 +135,8 @@
     <axis xyz="0 0 1"/>
     <limit lower="-0.3" upper="0.5" effort="10.0" velocity="10.0" />
-    <parent link="link2"/>
-    <child link="link3"/>
-  </joint>
-  <link name="link3">
+    <parent link="tl_2"/>
+    <child link="tl_3"/>
+  </joint>
+  <link name="tl_3">
     <inertial>
       <mass value="0.1"/>
@@ -161,8 +161,8 @@
     <axis xyz="0 0 1"/>
     <limit lower="-1.57" upper="1.57" effort="10.0" velocity="10.0" />
-    <parent link="link3"/>
-    <child link="link4"/>
-  </joint>
-  <link name="link4">
+    <parent link="tl_3"/>
+    <child link="tl_4"/>
+  </joint>
+  <link name="tl_4">
     <inertial>
       <mass value="0.1"/>
@@ -187,8 +187,8 @@
     <axis xyz="0 0 1"/>
     <limit lower="-0.5" upper="5.14" effort="10.0" velocity="10.0" />
-    <parent link="link4"/>
-    <child link="link5"/>
-  </joint>
-  <link name="link5">
+    <parent link="tl_4"/>
+    <child link="tl_5"/>
+  </joint>
+  <link name="tl_5">
     <inertial>
       <mass value="0.1"/>
@@ -213,8 +213,8 @@
     <axis xyz="0 0 1"/>
     <limit lower="-3.0" upper="2.9" effort="10.0" velocity="10.0" />
-    <parent link="link5"/>
-    <child link="link6"/>
-  </joint>
-  <link name="link6">
+    <parent link="tl_5"/>
+    <child link="tl_6"/>
+  </joint>
+  <link name="tl_6">
     <inertial>
       <mass value="0.1"/>
@@ -237,6 +237,6 @@
   <joint name="Irp6ottfgJoint1" type="prismatic">
     <origin rpy="0 0 0" xyz="0.0 0.0 0.15"/>
-    <parent link="link6"/>
-    <child link="gripper_link_1"/>
+    <parent link="tl_6"/>
+    <child link="tl_g1"/>
     <axis xyz="0 1 0" />
     <limit upper="0.1" lower="0" effort="10" velocity=".53" />
@@ -244,11 +244,11 @@
   <joint name="Irp6ottfgJoint1a" type="prismatic">
     <origin rpy="0 0 0" xyz="0.0 0.0 0.15"/>
-    <parent link="link6"/>
-    <child link="gripper_link_2"/>
+    <parent link="tl_6"/>
+    <child link="tl_g2"/>
     <axis xyz="0 -1 0" />
     <limit upper="0.1" lower="0" effort="10" velocity=".53" />
     <mimic joint="Irp6ottfgJoint1" />
   </joint>
-  <link name="gripper_link_1">
+  <link name="tl_g1">
     <inertial>
       <mass value="0.1"/>
@@ -269,5 +269,5 @@
     </collision>
   </link>
-<link name="gripper_link_2">
+<link name="tl_g2">
     <inertial>
       <mass value="0.1"/>
@@ -292,7 +292,7 @@
     <origin rpy="0 0 0.0" xyz="0.0 2.11 0.0"/>
     <parent link="world"/>
-    <child link="base_link_p"/>
-  </joint>
-  <link name="base_link_p">
+    <child link="pl_base"/>
+  </joint>
+  <link name="pl_base">
     <inertial>
       <mass value="0" />
@@ -322,8 +322,8 @@
     <axis xyz="0 0 1"/>
     <limit lower="-2.96705973" upper="2.96705973" effort="10.0" velocity="10.0" />
-    <parent link="base_link_p"/>
-    <child link="link1_p"/>
-  </joint>
-  <link name="link1_p">
+    <parent link="pl_base"/>
+    <child link="pl_1"/>
+  </joint>
+  <link name="pl_1">
     <inertial>
       <mass value="0.1"/>
@@ -349,8 +349,8 @@
     <axis xyz="0 0 1"/>
     <limit lower="-1.8" upper="-0.872664626" effort="10.0" velocity="10.0" />
-    <parent link="link1_p"/>
-    <child link="link2_p"/>
-  </joint>
-  <link name="link2_p">
+    <parent link="pl_1"/>
+    <child link="pl_2"/>
+  </joint>
+  <link name="pl_2">
     <inertial>
       <mass value="0.1"/>
@@ -375,8 +375,8 @@
     <axis xyz="0 0 1"/>
     <limit lower="-0.3" upper="0.5" effort="10.0" velocity="10.0" />
-    <parent link="link2_p"/>
-    <child link="link3_p"/>
-  </joint>
-  <link name="link3_p">
+    <parent link="pl_2"/>
+    <child link="pl_3"/>
+  </joint>
+  <link name="pl_3">
     <inertial>
       <mass value="0.1"/>
@@ -401,8 +401,8 @@
     <axis xyz="0 0 1"/>
     <limit lower="-1.57" upper="1.57" effort="10.0" velocity="10.0" />
-    <parent link="link3_p"/>
-    <child link="link4_p"/>
-  </joint>
-  <link name="link4_p">
+    <parent link="pl_3"/>
+    <child link="pl_4"/>
+  </joint>
+  <link name="pl_4">
     <inertial>
       <mass value="0.1"/>
@@ -427,8 +427,8 @@
     <axis xyz="0 0 1"/>
     <limit lower="-0.5" upper="5.14" effort="10.0" velocity="10.0" />
-    <parent link="link4_p"/>
-    <child link="link5_p"/>
-  </joint>
-  <link name="link5_p">
+    <parent link="pl_4"/>
+    <child link="pl_5"/>
+  </joint>
+  <link name="pl_5">
     <inertial>
       <mass value="0.1"/>
@@ -453,8 +453,8 @@
     <axis xyz="0 0 1"/>
     <limit lower="-3.0" upper="2.9" effort="10.0" velocity="10.0" />
-    <parent link="link5_p"/>
-    <child link="link6_p"/>
-  </joint>
-  <link name="link6_p">
+    <parent link="pl_5"/>
+    <child link="pl_6"/>
+  </joint>
+  <link name="pl_6">
     <inertial>
       <mass value="0.1"/>
@@ -477,6 +477,6 @@
   <joint name="Irp6ptfgJoint1" type="prismatic">
     <origin rpy="0 0 0" xyz="0.0 0.0 0.15"/>
-    <parent link="link6_p"/>
-    <child link="gripper_link_p_1"/>
+    <parent link="pl_6"/>
+    <child link="pl_g1"/>
     <axis xyz="0 1 0" />
     <limit upper="0.1" lower="0" effort="10" velocity=".53" />
@@ -484,11 +484,11 @@
   <joint name="Irp6ptfgJoint1a" type="prismatic">
     <origin rpy="0 0 0" xyz="0.0 0.0 0.15"/>
-    <parent link="link6_p"/>
-    <child link="gripper_link_p_2"/>
+    <parent link="pl_6"/>
+    <child link="pl_g2"/>
     <axis xyz="0 -1 0" />
     <limit upper="0.1" lower="0" effort="10" velocity=".53" />
     <mimic joint="Irp6ptfgJoint1" />
   </joint>
-  <link name="gripper_link_p_1">
+  <link name="pl_g1">
     <inertial>
       <mass value="0.1"/>
@@ -509,5 +509,5 @@
     </collision>
   </link>
-<link name="gripper_link_p_2">
+<link name="pl_g2">
     <inertial>
       <mass value="0.1"/>

Commit message: irp6 urdf update - track camera

File: irp6_description/robots/irp6pboth.urdf.xacro (robot description, xacro)
@@ -288,4 +288,11 @@
     </collision>
   </link>
+<joint name="tl_camera" type="fixed">
+    <origin rpy="0.0 0.0 1.57" xyz="-0.0551 0.0 0.13"/>
+    <parent link="tl_6"/>
+    <child link="t_c"/>
+  </joint>
+<link name="t_c">
+</link>
 <!-- -.-.-.-.-.-.-.-.-.-.-.-.-.-.-.-.-.-.-.-.-.-.-.-.-.-.-.-.-.-.-.-.-.-.-.-.-.-.-.-.-.-.- -->
   <joint name="base_joint_p" type="fixed">

Commit message: irp6 urdf update - postument camera

File: irp6_description/robots/irp6pboth.urdf.xacro (robot description, xacro)
@@ -295,4 +295,11 @@
 <link name="t_c">
 </link>
+<joint name="tl_camera_optical_frame" type="fixed">
+    <origin rpy="0.0 0.0 3.14" xyz="0.0 0.0 0.0"/>
+    <parent link="t_c"/>
+    <child link="t_c_optical_frame"/>
+  </joint>
+<link name="t_c_optical_frame">
+</link>
 <!-- -.-.-.-.-.-.-.-.-.-.-.-.-.-.-.-.-.-.-.-.-.-.-.-.-.-.-.-.-.-.-.-.-.-.-.-.-.-.-.-.-.-.- -->
   <joint name="base_joint_p" type="fixed">
@@ -535,4 +542,18 @@
     </collision>
   </link>
+<joint name="pl_camera" type="fixed">
+    <origin rpy="0.0 0.0 -1.57" xyz="0.0551 0.0 0.13"/>
+    <parent link="pl_6"/>
+    <child link="p_c"/>
+  </joint>
+<link name="p_c">
+</link>
+<joint name="pl_camera_optical_frame" type="fixed">
+    <origin rpy="0.0 0.0 3.14" xyz="0.0 0.0 0.0"/>
+    <parent link="p_c"/>
+    <child link="p_c_optical_frame"/>
+  </joint>
+<link name="p_c_optical_frame">
+</link>
 <!-- Kinect                       -->
 <!--

Commit message: xacro fix

File: irp6_description/robots/irp6pboth.urdf.xacro (robot description, xacro)
@@ -6,4 +6,10 @@
        xmlns:interface="http://playerstage.sourceforge.net/gazebo/xmlschema/#interface">
   <xacro:property name="M_PI" value="3.14159"/>
+    <material name="orange">
+      <color rgba=".99 .4 .1 1" />
+    </material>
+    <material name="silver">
+      <color rgba=".8 .8 .8 1" />
+    </material>
   <link name="world">
     <!--<inertial>
@@ -36,7 +42,5 @@
       <box size=".462 1.609 .25" />
     </geometry>
-    <material name="gray">
-      <color rgba=".2 .2 .2 1" />
-    </material>
+    <material name="orange"/>
   </visual>
   <collision>
@@ -58,7 +62,5 @@
       <box size="0.4 0.4 0.15" />
     </geometry>
-    <material name="gray">
-      <color rgba=".2 .2 .2 1" />
-    </material>
+    <material name="orange"/>
   </visual>
   <collision>
@@ -94,4 +96,5 @@
         <mesh filename="package://irp6_description/meshes/link1.3ds" />
       </geometry>
+      <material name="orange"/>
     </visual>
     <collision>
@@ -259,4 +262,5 @@
          <box size="0.05 0.04 0.12" />
       </geometry>
+      <material name="silver"/>
     </visual>
     <collision>
@@ -278,4 +282,5 @@
          <box size="0.05 0.04 0.12" />
       </geometry>
+      <material name="silver"/>
     </visual>
     <collision>
@@ -348,7 +353,5 @@
         <box size="0.4 0.4 0.4" />
       </geometry>
-      <material name="gray">
-      <color rgba=".2 .2 .2 1" />
-    </material>
+      <material name="orange"/>
   </visual>
   </link>
@@ -371,4 +374,5 @@
         <mesh filename="package://irp6_description/meshes/link1.3ds" />
       </geometry>
+       <material name="orange"/>
     </visual>
     <collision>
@@ -536,4 +540,5 @@
          <box size="0.05 0.04 0.12" />
       </geometry>
+      <material name="silver"/>
     </visual>
     <collision>
@@ -554,5 +559,6 @@
       <geometry>
          <box size="0.05 0.04 0.12" />
-      </geometry>origin
+      </geometry>
+      <material name="silver"/>
     </visual>
     <collision>

Commit message: fixed conveyor added to urdf

File: irp6_description/robots/irp6pboth.urdf.xacro (robot description, xacro)
@@ -27,8 +27,32 @@
     </collision>
   </link>
-  <joint name="base_joint" type="fixed">
+  <joint name="t_base_joint" type="fixed">
     <parent link="world"/>
     <child link="tl_base"/>
   </joint>
+  <joint name="conv_base_joint" type="fixed">
+    <parent link="world"/>
+    <child link="conveyor"/>
+  </joint>
+<link name="conveyor">
+  <inertial>
+    <mass value="1"/>
+    <inertia ixx="100" ixy="0" ixz="0" iyy="100" iyz="0" izz="100" />
+    <origin xyz="0 0 0"/>
+  </inertial>
+  <visual>
+    <origin xyz="0.5 1 0.0" />
+    <geometry>
+      <mesh filename="package://irp6_description/meshes/conveyor.3ds" />
+    </geometry>
+    <material name="orange"/>
+  </visual>
+  <collision>
+    <origin xyz="0 0 0" />
+    <geometry>
+      <box size=".0 .0 .0" />
+    </geometry>
+  </collision>
+</link>
 <link name="tl_base">
   <inertial>

Commit message: fixed new wrist in urdf and 3ds

File: irp6_description/robots/irp6pboth.urdf.xacro (robot description, xacro)
@@ -248,5 +248,5 @@
     </inertial>
     <visual>
-      <origin rpy="0 0 0.0" xyz="0 0.0 0.15"/>
+      <origin rpy="0 0 0.0" xyz="0 0.0 0.105"/>
       <geometry>
          <mesh filename="package://irp6_description/meshes/link6.3ds" />
@@ -526,5 +526,5 @@
     </inertial>
     <visual>
-      <origin rpy="0 0 0.0" xyz="0 0.0 0.15"/>
+      <origin rpy="0 0 0.0" xyz="0 0.0 0.105"/>
       <geometry>
          <mesh filename="package://irp6_description/meshes/link6.3ds" />

Commit message: conveyor visualisation fix

File: irp6_description/robots/irp6pboth.urdf.xacro (robot description, xacro)
@@ -42,5 +42,5 @@
   </inertial>
   <visual>
-    <origin xyz="0.5 1 0.0" />
+    <origin xyz="0.59 0.7 0.0" />
     <geometry>
       <mesh filename="package://irp6_description/meshes/conveyor.3ds" />

Commit message: urdf dimensions corrections

File: irp6_description/robots/irp6pboth.urdf.xacro (robot description, xacro)
@@ -42,5 +42,5 @@
   </inertial>
   <visual>
-    <origin xyz="0.59 0.7 0.0" />
+    <origin xyz="0.59 0.45 0.0" />
     <geometry>
       <mesh filename="package://irp6_description/meshes/conveyor.3ds" />
@@ -64,12 +64,12 @@
     <origin xyz="0 .6045 .125" />
     <geometry>
-      <box size=".462 1.609 .25" />
+      <box size=".48 2.0 .25" />
     </geometry>
     <material name="orange"/>
   </visual>
   <collision>
-    <origin xyz="0 .6045 .07" />
+    <origin xyz="0 .6045 .125" />
     <geometry>
-      <box size=".462 1.609 .2" />
+      <box size=".48 2.0 .25" />
     </geometry>
   </collision>
